File: transistor matcher/transistor_matcher/transistor_matcher.kicad_pcb (KiCad board)
At the start: 2 copper layers, 99.1 x 69.9 mm, 15 parts, among them J1 Conn_02x05_Odd_Even, Q1 Q_NPN_BCE, Q2 Q_NPN_BCE, Q3 Q_PNP_BCE, Q4 Q_PNP_BCE

Commit message: Updates to transistor matcher
Parts:
- Q1, Q2, Q3, Q4: footprint Connector_PinHeader_1.00mm:PinHeader_1x03_P1.00mm_Vertical -> Package_TO_SOT_THT:TO-92L_Inline_Wide
- TP1, TP2: footprint Connector_PinHeader_1.00mm:PinHeader_1x02_P1.00mm_Vertical -> Connector_PinHeader_2.54mm:PinHeader_1x02_P2.54mm_Vertical
- moved D1 17.8 mm to (141.7, 111.1)
- moved D2 17.8 mm to (146.7, 103.5)
- moved R1 17.8 mm to (136.6, 103.5)
- moved R4 17.8 mm to (151.8, 103.5)
- moved R5 10.2 mm to (174.7, 118.7)
- moved R2 10.2 mm to (112.4, 118.7)
- moved R3 9.67 mm to (115.0, 118.7)
- moved R6 9.67 mm to (177.2, 118.7)
- moved Q2 7.73 mm to (120.1, 76.8), turned to 270 degrees
- moved Q4 7.73 mm to (182.3, 76.8), turned to 270 degrees
- moved Q1 7.62 mm to (107.4, 76.8), turned to 270 degrees
- moved Q3 7.62 mm to (169.6, 76.8), turned to 270 degrees
- moved TP2 5.09 mm to (174.7, 100.9)
- moved TP1 5.08 mm to (112.4, 100.9)
Routing:
- net -12V: track 82.9 -> 45.1 mm
- net Net-(D2-Pad1): track 34.4 -> 49.3 mm
- net Net-(D1-Pad2): track 34.4 -> 48.7 mm
- net Net-(Q1-Pad3): track 20.0 -> 31.3 mm
- net Net-(Q4-Pad3): track 20.0 -> 31.3 mm
- net Net-(Q3-Pad3): track 20.2 -> 31.3 mm
- net Net-(Q2-Pad3): track 20.2 -> 31.3 mm
- net +12V: track 68.6 -> 58.1 mm
Other:
- net class Default: clearance 0.2 -> 0.5
- rule trace_clearance: 0.2 -> 0.5
- board text added: "+12"
- board text added: "-12v"
- board text added: "B C E"
- board text added: "GND GND GND"
- board text added: "NPN"
- board text added: "PNP"
- board text added: "Transistor Matcher"
